Commit message: Tow URDF, base rscorbot and scorbot as printer

File: src/scorbot_er_v/urdf/scorbot_base.urdf (robot description, URDF)
Before this commit: robot scorbot-er-v-plus, 9 links, 8 joints
Links:
- removed link extruder_link
- link base_link: mass 24.144 -> 54.14
- link body_link: mass 4.1847 -> 4.26
- link elbow_link: mass 1.3299 -> 1.33
- link roll_wrist_link: mass 0.3891 -> 0.208
- link shoulder_link: mass 2.1816 -> 2.16
- link slide_base_link: mass 5.7681 -> 5.77
- link wrist_link: mass 0.11142 -> 0.11
Joints:
- removed joint extruder_screw_joint
- removed joint world_joint
- added joint world_link: type fixed, parent world, child base_link
- joint body_joint: origin xyz=0 0.354 0 rpy=1.5708 -1.5708 0 -> xyz=0 0.354 0 rpy=-1.570796327 -1.570796327 0
- joint elbow_joint: axis 0 0 -1 -> 0 0 1
- joint roll_wrist_joint: origin xyz=0 0 0 rpy=1.5708 0 0 -> xyz=0 0 0 rpy=1.5707963267949 0 0
- joint shoulder_joint: axis 0 0 -1 -> 0 0 1; origin xyz=0.025 0 0 rpy=1.5708 0 0 -> xyz=0.025 0 0 rpy=1.570796327 0 0
- joint slide_base_joint: limit lower=0 upper=0.9 effort=0 velocity=0 -> lower=0 upper=0.950 effort=0 velocity=0; origin xyz=0 0.17 0.096 rpy=1.5708 0 3.1416 -> xyz=0 0.17 0.096 rpy=1.570796327 0 3.141592654
- joint wrist_joint: axis 0 0 -1 -> 0 0 1; origin xyz=0.22 0 0 rpy=0 0 1.5708 -> xyz=0.22 0 0 rpy=0 0 1.5707963267949

File: src/scorbot_er_v/urdf/scorbot_printer.urdf (robot description, URDF)
Before this commit: robot scorbot-er-v-plus, 8 links, 7 joints
Links:
- added link extruder_link, mass 0.00058199; collision mesh filename=package://scorbot_er_v/meshes-extruder/extruder_link.STL; visual mesh filename=package://scorbot_er_v/meshes-extruder/extruder_link.STL
- link base_link: mass 54.14 -> 24.144; geometry collision mesh filename=package://scorbot_er_v/meshes-extruder/slide_base_link.STL; visual mesh filename=package://scorbot_er_v/meshes-extruder/slide_base_link.STL
- link body_link: mass 4.26 -> 4.1847; geometry collision mesh filename=package://scorbot_er_v/meshes-extruder/body_link.STL; visual mesh filename=package://scorbot_er_v/meshes-extruder/body_link.STL
- link elbow_link: mass 1.33 -> 1.3299; geometry collision mesh filename=package://scorbot_er_v/meshes-extruder/elbow_link.STL; visual mesh filename=package://scorbot_er_v/meshes-extruder/elbow_link.STL
- link roll_wrist_link: mass 0.208 -> 0.3891; geometry collision mesh filename=package://scorbot_er_v/meshes-extruder/roll_wrist_link.STL; visual mesh filename=package://scorbot_er_v/meshes-extruder/roll_wrist_link.STL
- link shoulder_link: mass 2.16 -> 2.1816; geometry collision mesh filename=package://scorbot_er_v/meshes-extruder/shoulder_link.STL; visual mesh filename=package://scorbot_er_v/meshes-extruder/shoulder_link.STL
- link slide_base_link: mass 5.77 -> 5.7681; geometry collision mesh filename=package://scorbot_er_v/meshes-extruder/base_link.STL; visual mesh filename=package://scorbot_er_v/meshes-extruder/base_link.STL
- link wrist_link: mass 0.11 -> 0.11142; geometry collision mesh filename=package://scorbot_er_v/meshes-extruder/wrist_link.STL; visual mesh filename=package://scorbot_er_v/meshes-extruder/wrist_link.STL
Joints:
- removed joint world_link
- added joint extruder_screw_joint: type continuous, parent roll_wrist_link, child extruder_link, origin xyz=0 0.011037 0.126 rpy=1.5708 -1.5708 0, axis 0 0 1
- added joint world_joint: type fixed, parent world, child base_link
- joint body_joint: origin xyz=0 0.354 0 rpy=-1.570796327 -1.570796327 0 -> xyz=0 0.354 0 rpy=1.5708 -1.5708 0
- joint elbow_joint: axis 0 0 1 -> 0 0 -1
- joint roll_wrist_joint: origin xyz=0 0 0 rpy=1.5707963267949 0 0 -> xyz=0 0 0 rpy=1.5708 0 0
- joint shoulder_joint: axis 0 0 1 -> 0 0 -1; origin xyz=0.025 0 0 rpy=1.570796327 0 0 -> xyz=0.025 0 0 rpy=1.5708 0 0
- joint slide_base_joint: limit lower=0 upper=0.950 effort=0 velocity=0 -> lower=0 upper=0.9 effort=0 velocity=0; origin xyz=0 0.17 0.096 rpy=1.570796327 0 3.141592654 -> xyz=0 0.17 0.096 rpy=1.5708 0 3.1416
- joint wrist_joint: axis 0 0 1 -> 0 0 -1; origin xyz=0.22 0 0 rpy=0 0 1.5707963267949 -> xyz=0.22 0 0 rpy=0 0 1.5708
