Commit message: Fix meshes path

File: src/scorbot_er_v/urdf/scorbot_printer.urdf (robot description, URDF)
Before this commit: robot scorbot-er-v-plus, 9 links, 8 joints
Links:
- link base_link: geometry collision mesh filename=package://scorbot_er_v/meshes/slide_base_link.STL; visual mesh filename=package://scorbot_er_v/meshes/slide_base_link.STL
- link body_link: geometry collision mesh filename=package://scorbot_er_v/meshes/body_link.STL; visual mesh filename=package://scorbot_er_v/meshes/body_link.STL
- link elbow_link: geometry collision mesh filename=package://scorbot_er_v/meshes/elbow_link.STL; visual mesh filename=package://scorbot_er_v/meshes/elbow_link.STL
- link extruder_link: geometry collision mesh filename=package://scorbot_er_v/meshes/extruder_link.STL; visual mesh filename=package://scorbot_er_v/meshes/extruder_link.STL
- link roll_wrist_link: geometry collision mesh filename=package://scorbot_er_v/meshes/roll_wrist_link.STL; visual mesh filename=package://scorbot_er_v/meshes/roll_wrist_link.STL
- link shoulder_link: geometry collision mesh filename=package://scorbot_er_v/meshes/shoulder_link.STL; visual mesh filename=package://scorbot_er_v/meshes/shoulder_link.STL
- link slide_base_link: geometry collision mesh filename=package://scorbot_er_v/meshes/base_link.STL; visual mesh filename=package://scorbot_er_v/meshes/base_link.STL
- link wrist_link: geometry collision mesh filename=package://scorbot_er_v/meshes/wrist_link.STL; visual mesh filename=package://scorbot_er_v/meshes/wrist_link.STL
Joints:
- joint body_joint: axis 0 0 1 -> 0 0 -1

Commit message: Fix axis and meshes orientations

File: src/scorbot_er_v/urdf/scorbot_printer.urdf (robot description, URDF)
Before this commit: robot scorbot-er-v-plus, 9 links, 8 joints
Joints:
- joint body_joint: axis 0 0 -1 -> 0 0 1; origin xyz=0 0.354 0 rpy=1.5708 -1.5708 0 -> xyz=0 0.354 0 rpy=-1.5708 -1.5708 0
- joint extruder_screw_joint: origin xyz=0 0.011037 0.126 rpy=1.5708 -1.5708 0 -> xyz=0 -0.011037 0.126 rpy=-1.5708 3.1416 0

Commit message: Fix axis rotation

File: src/scorbot_er_v/urdf/scorbot_printer.urdf (robot description, URDF)
Before this commit: robot scorbot-er-v-plus, 9 links, 8 joints
Joints:
- joint elbow_joint: axis 0 0 -1 -> 0 0 1
- joint shoulder_joint: axis 0 0 -1 -> 0 0 1
- joint wrist_joint: axis 0 0 -1 -> 0 0 1

Commit message: Add the hotend link

File: src/scorbot_er_v/urdf/scorbot_printer.urdf (robot description, URDF)
Before this commit: robot scorbot-er-v-plus, 9 links, 8 joints
Links:
- added link hotend_link
Joints:
- added joint hotend_joint: type fixed, parent roll_wrist_link, child hotend_link, origin xyz=-0.049 -0.0137 0.132 rpy=0 -1.5708 0
